File: mm_motor_control.kicad_sch (KiCad schematic)
At the start: 0 parts

Commit message: tp2
Parts:
- added C20: 10nF, Capacitor_SMD:C_0603_1608Metric, symbol Device:C
- added C30: 22nF, Capacitor_SMD:C_0603_1608Metric, symbol Device:C
- added C31: 2.2uF, Capacitor_SMD:C_0603_1608Metric, symbol Device:C
- added C32: 22uF, Capacitor_SMD:C_0603_1608Metric, symbol Device:C
- added C34: 1nF, Capacitor_SMD:C_0603_1608Metric, symbol Device:C
- added C9: 1uF, Capacitor_SMD:C_0603_1608Metric, symbol Device:C
- added R51, R52: 18k, Resistor_SMD:R_0603_1608Metric, symbol Device:R
- added R53: 15k, Resistor_SMD:R_0603_1608Metric, symbol Device:R
- added R54: 2k, Resistor_SMD:R_0603_1608Metric, symbol Device:R
- added R55: 1k, Resistor_SMD:R_0603_1608Metric, symbol Device:R
- added R56: 47k, Resistor_SMD:R_0603_1608Metric, symbol Device:R
- added R57, R58: 330m, Resistor_SMD:R_2512_6332Metric, symbol Device:R
- added U2: STSPIN240, Package_DFN_QFN:VQFN-16-1EP_3x3mm_P0.5mm_EP1.8x1.8mm, symbol Driver_Motor:STSPIN240
Connections:
- net EN: now also R51.1
- net FAULT: now also C20.1, R51.2, U2.13 (EN/FLT)
- net OUT_A1: now also U2.3 (OUTA1)
- net OUT_A2: now also U2.5 (OUTA2)
- net OUT_B1: now also U2.10 (OUTB1)
- net OUT_B2: now also U2.8 (OUTB2)
- net PHASE_A: now also U2.1 (PHA)
- net PHASE_B: now also U2.15 (PHB)
- net PWM_A: now also U2.2 (PWMA)
- net PWM_B: now also U2.16 (PWMB)
- net STBY/RESET: now also C34.1, R52.2, U2.14 (STBY/RESET)
- new net: R55.1, R56.1, U2.12 (TOFF)
- new net: C9.1, R53.2, R54.1, U2.11 (REF)
- new net: R57.1, U2.4 (SENSEA)
- new net: R58.1, U2.9 (SENSEB)
- new net: C30.1, R55.2
- new net +3.3V: R53.1
- new net +BATT: C31.1, C32.1, R52.1, U2.6 (VS)
- new net GND: C20.2, C30.2, C31.2, C32.2, C34.2, C9.2, R54.2, R56.2, R57.2, R58.2, U2.17 (EPAD), U2.7 (GND)
