File: mm_power.kicad_sch (KiCad schematic)
At the start: 1 part, among them J5 Conn_01x02

Commit message: tp2
Parts:
- added C7, C8: 22uF, Capacitor_SMD:C_0603_1608Metric, symbol Device:C
- added D1: 1N4003, Diode_THT:D_DO-41_SOD81_P10.16mm_Horizontal, symbol Diode:1N4003
- added R10: 180, Resistor_SMD:R_0603_1608Metric, symbol Device:R
- added U3: LP5907MFX-3.3, Package_TO_SOT_SMD:SOT-23-5, symbol Regulator_Linear:LP5907MFX-3.3
Connections:
- net +BATT: now also C7.1, U3.1 (IN), U3.3 (EN)
- net GND: now also C7.2, C8.2, D1.1 (K), U3.2 (GND)
- new net: D1.2 (A), R10.2
- new net +3.3V: C8.1, R10.1, U3.5 (OUT)
